File: ELECTRONICS/main_board.sch (EAGLE design)
At the start: 18 parts, among them CON3 Accelerometer connector, CON4 UART connector, IC1 LM324D, IC2 7414N

Commit message: Some edits.
Parts:
- CON2: device con-lstb:MA20-2 -> con-lstb:MA18-2
- LED1: value (none) -> Power indicator
Connections:
- net ADC_CS: now also CON3.4; no longer CON3.1
- net ADC_DOUT: now also CON3.1; no longer CON3.2
- net ADC_SCLK: now also CON3.2; no longer CON3.4
- net GND: no longer CON2.39
Changed lines of the file:
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@@
 <layer number="48" name="Document" color="7" fill="1" visible="yes" active="no"/>
 <layer number="49" name="Reference" color="7" fill="1" visible="yes" active="no"/>
-<layer number="51" name="tDocu" color="6" fill="1" visible="yes" active="no"/>
+<layer number="51" name="tDocu" color="7" fill="1" visible="yes" active="no"/>
 <layer number="52" name="bDocu" color="7" fill="1" visible="yes" active="no"/>
 <layer number="90" name="Modules" color="5" fill="1" visible="yes" active="yes"/>
@@
 <part name="IC2" library="74xx-eu" deviceset="74*14" device="N" value="7414N"/>
 <part name="R1" library="rcl" deviceset="R-EU_" device="R0805" value="100K"/>
-<part name="CON2" library="con-lstb" deviceset="MA20-2" device=""/>
+<part name="CON2" library="con-lstb" deviceset="MA18-2" device=""/>
 <part name="CON1" library="con-lstb" deviceset="MA05-2" device=""/>
 <part name="R2" library="rcl" deviceset="R-EU_" device="R0805" value="100K"/>
@@
 <part name="C1" library="rcl" deviceset="C-EU" device="C0805K" value="100nF"/>
 <part name="C2" library="rcl" deviceset="C-EU" device="C0805K" value="100nF"/>
-<part name="LED1" library="led" deviceset="LED" device="CHIP-LED0805"/>
+<part name="LED1" library="led" deviceset="LED" device="CHIP-LED0805" value="Power indicator"/>
 <part name="R4" library="rcl" deviceset="R-EU_" device="R0805" value="100R"/>
 <part name="GND9" library="supply1" deviceset="GND" device=""/>
@@
 <part name="R5" library="rcl" deviceset="R-EU_" device="R0805" value="50R"/>
 <part name="CON4" library="con-molex" deviceset="22-?-04" device="27-2041" value="UART connector"/>
-<part name="FRAME3" library="frames" deviceset="A4L-LOC" device=""/>
+<part name="FRAME3" library="frames" deviceset="A4L-LOC" device="" value="Main board"/>
 <part name="C3" library="rcl" deviceset="C-EU" device="C1206K" value="10uF"/>
 <part name="GND7" library="supply1" deviceset="GND" device=""/>
@@
 <instance part="IC2" gate="F" x="238.76" y="43.18"/>
 <instance part="R1" gate="G$1" x="86.36" y="121.92" rot="R90"/>
-<instance part="CON2" gate="G$1" x="58.42" y="45.72" rot="R180"/>
+<instance part="CON2" gate="G$1" x="58.42" y="50.8" rot="R180"/>
 <instance part="CON1" gate="G$1" x="33.02" y="137.16" rot="R180"/>
 <instance part="R2" gate="G$1" x="86.36" y="137.16" rot="R90"/>
@@
 <pinref part="GND3" gate="1" pin="GND"/>
 <pinref part="CON2" gate="G$1" pin="25"/>
-<wire x1="48.26" y1="40.64" x2="48.26" y2="22.86" width="0.1524" layer="91"/>
-<wire x1="48.26" y1="22.86" x2="48.26" y2="20.32" width="0.1524" layer="91"/>
+<wire x1="48.26" y1="40.64" x2="48.26" y2="20.32" width="0.1524" layer="91"/>
 <wire x1="50.8" y1="40.64" x2="48.26" y2="40.64" width="0.1524" layer="91"/>
 <junction x="48.26" y="40.64"/>
-<pinref part="CON2" gate="G$1" pin="39"/>
-<wire x1="50.8" y1="22.86" x2="48.26" y2="22.86" width="0.1524" layer="91"/>
-<junction x="48.26" y="22.86"/>
 </segment>
 <segment>
@@
 </segment>
 <segment>
-<pinref part="CON3" gate="1" pin="2"/>
-<wire x1="121.92" y1="63.5" x2="106.68" y2="63.5" width="0.1524" layer="91"/>
-<label x="106.68" y="63.5" size="1.778" layer="95"/>
+<pinref part="CON3" gate="1" pin="1"/>
+<wire x1="137.16" y1="63.5" x2="154.94" y2="63.5" width="0.1524" layer="91"/>
+<label x="142.24" y="63.5" size="1.778" layer="95"/>
 </segment>
 </net>
@@
 <pinref part="CON3" gate="1" pin="3"/>
 <wire x1="137.16" y1="66.04" x2="154.94" y2="66.04" width="0.1524" layer="91"/>
-<label x="144.78" y="66.04" size="1.778" layer="95"/>
+<label x="142.24" y="66.04" size="1.778" layer="95"/>
 </segment>
 </net>
@@
 </segment>
 <segment>
-<pinref part="CON3" gate="1" pin="1"/>
-<wire x1="137.16" y1="63.5" x2="154.94" y2="63.5" width="0.1524" layer="91"/>
-<label x="144.78" y="63.5" size="1.778" layer="95"/>
+<pinref part="CON3" gate="1" pin="4"/>
+<wire x1="121.92" y1="66.04" x2="109.22" y2="66.04" width="0.1524" layer="91"/>
+<label x="109.22" y="66.04" size="1.778" layer="95"/>
 </segment>
 </net>
@@
 </segment>
 <segment>
-<pinref part="CON3" gate="1" pin="4"/>
-<wire x1="121.92" y1="66.04" x2="106.68" y2="66.04" width="0.1524" layer="91"/>
-<label x="106.68" y="66.04" size="1.778" layer="95"/>
-</segment>
-</net>
+<pinref part="CON3" gate="1" pin="2"/>
+<wire x1="121.92" y1="63.5" x2="109.22" y2="63.5" width="0.1524" layer="91"/>
+<label x="109.22" y="63.5" size="1.778" layer="95"/>
+</segment>
+</net>
