File: ELECTRONICS/accelerometer_board.brd (EAGLE design)
At the start: 33 x 21 mm, 13 parts, among them CON1 Main board connector, IC3 AD7887BRZ, IC4 ADXL203CE

Commit message: Accelerometer PCB is finish! :)
Parts:
- moved C3 3.69 mm to (22.2, 16.6)
- moved C6 3.69 mm to (28.1, 8.98)
- moved IC3 3.69 mm to (17.7, 14.4)
- moved LED1 3.69 mm to (25.5, 6.21)
- moved C5 3.69 mm to (16.7, 8.19)
- moved R3 3.69 mm to (15.9, 20.1)
- moved C1 3.69 mm to (13.9, 7.02)
- moved R1 3.69 mm to (20.8, 6.21)
- moved C2 3.69 mm to (27.6, 11.2)
- moved C4 3.69 mm to (22.3, 12.8)
- moved IC4 3.69 mm to (26.6, 15.3)
- moved R2 3.69 mm to (30.9, 15.0)
- moved CON1 3.37 mm to (7.53, 13.8)
Routing:
- net ADC_DOUT: track 10.1 -> 10.7 mm
Other:
- board size 33 x 21 mm -> 36 x 28 mm
- board text removed: "OBS! Check connectors and via sizes! As well as component dimensions"

Commit message: Final PCB
Parts:
- renumbered IC3 to IC1, IC4 to IC2
Changed lines of the file:
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@@
 <attribute name="VALUE" x="1.9144" y="21.9818" size="0.8128" layer="27" ratio="10"/>
 </element>
-<element name="IC3" library="tobylib" package="SO08" value="AD7887BRZ" x="17.7386" y="14.438" smashed="yes">
+<element name="IC1" library="tobylib" package="SO08" value="AD7887BRZ" x="17.7386" y="14.438" smashed="yes">
 <attribute name="VALUE" x="20.8374" y="18.5274" size="0.8128" layer="27" ratio="10" rot="R180"/>
 <attribute name="NAME" x="14.7668" y="13.7268" size="0.8128" layer="25" ratio="10" rot="R90"/>
 </element>
-<element name="IC4" library="tobylib" package="LCC127P500X500X220-8N" value="ADXL203CE" x="26.5778" y="15.3016" smashed="yes" rot="R180">
+<element name="IC2" library="tobylib" package="LCC127P500X500X220-8N" value="ADXL203CE" x="26.5778" y="15.3016" smashed="yes" rot="R180">
 <attribute name="PACKAGE" value="CLCC-8 Analog Devices" x="26.5778" y="15.3016" size="1.778" layer="27" rot="R180" display="off"/>
 <attribute name="AVAILABILITY" value="Good" x="26.5778" y="15.3016" size="1.778" layer="27" rot="R180" display="off"/>
@@
 <signals>
 <signal name="GND" class="1">
-<contactref element="IC3" pad="3"/>
-<contactref element="IC4" pad="3"/>
+<contactref element="IC1" pad="3"/>
+<contactref element="IC2" pad="3"/>
 <contactref element="LED1" pad="C"/>
 <contactref element="C5" pad="2"/>
@@
 </signal>
 <signal name="+3V3" class="1">
-<contactref element="IC3" pad="2"/>
+<contactref element="IC1" pad="2"/>
 <contactref element="C5" pad="1"/>
 <contactref element="C6" pad="1"/>
-<contactref element="IC4" pad="8"/>
+<contactref element="IC2" pad="8"/>
 <contactref element="C2" pad="1"/>
 <contactref element="R1" pad="2"/>
@@
 </signal>
 <signal name="N$5">
-<contactref element="IC4" pad="7"/>
+<contactref element="IC2" pad="7"/>
 <contactref element="C4" pad="1"/>
-<contactref element="IC3" pad="4"/>
+<contactref element="IC1" pad="4"/>
 <wire x1="24.5966" y1="14.0316" x2="22.479" y2="14.0316" width="0.4064" layer="1"/>
 <wire x1="22.479" y1="14.0316" x2="22.2598" y2="13.8124" width="0.4064" layer="1"/>
@@
 </signal>
 <signal name="ADC_CS">
-<contactref element="IC3" pad="1"/>
+<contactref element="IC1" pad="1"/>
 <contactref element="CON1" pad="4"/>
 <via x="13.5476" y="12.787" extent="1-16" drill="0.5" diameter="1.27" shape="octagon"/>
@@
 <signal name="ADC_DIN">
 <contactref element="CON1" pad="3"/>
-<contactref element="IC3" pad="6"/>
+<contactref element="IC1" pad="6"/>
 <wire x1="18.3736" y1="17.5114" x2="18.3736" y2="21.4738" width="0.4064" layer="1"/>
 <wire x1="18.3736" y1="21.4738" x2="17.51" y2="22.3374" width="0.4064" layer="1"/>
@@
 </signal>
 <signal name="ADC_SCLK">
-<contactref element="IC3" pad="8"/>
+<contactref element="IC1" pad="8"/>
 <contactref element="CON1" pad="2"/>
 <wire x1="13.3698" y1="16.6986" x2="13.3952" y2="16.724" width="0.4064" layer="16"/>
@@
 </signal>
 <signal name="N$8">
-<contactref element="IC4" pad="1"/>
+<contactref element="IC2" pad="1"/>
 <contactref element="R2" pad="2"/>
 <wire x1="30.9212" y1="14.0468" x2="28.5742" y2="14.0468" width="0.4064" layer="1"/>
@@
 <signal name="N$9">
 <contactref element="R3" pad="1"/>
-<contactref element="IC3" pad="7"/>
+<contactref element="IC1" pad="7"/>
 <wire x1="17.1036" y1="17.5114" x2="17.1036" y2="19.833" width="0.4064" layer="1"/>
 <wire x1="17.1036" y1="19.833" x2="16.809" y2="20.1276" width="0.4064" layer="1"/>
 </signal>
 <signal name="N$10">
-<contactref element="IC3" pad="5"/>
+<contactref element="IC1" pad="5"/>
 <contactref element="C3" pad="1"/>
-<contactref element="IC4" pad="6"/>
+<contactref element="IC2" pad="6"/>
 <wire x1="24.5966" y1="15.3016" x2="22.5298" y2="15.3016" width="0.4064" layer="1"/>
 <wire x1="22.5298" y1="15.3016" x2="22.2344" y2="15.597" width="0.4064" layer="1"/>
