File: ELECTRONICS/accelerometer_board.sch (EAGLE design)
At the start: 13 parts, among them IC3 AD7887BRZ, IC4 ADXL203CE

Commit message: Some edits.
Parts:
- CON1: value (none) -> Main board connector
- LED1: value (none) -> Power indicator
Connections:
- net N$3 renamed ADC_DIN
- removed net N$1: CON1.1, IC3.!CS
- removed net N$2: CON1.2, R3.2
- removed net N$4: CON1.4, IC3.SCLK
- removed net N$6: C3.1, IC3.AIN1, IC4.YOUT
- new net ADC_CS: CON1.4, IC3.!CS
- new net ADC_DOUT: CON1.1, R3.2
- new net ADC_SCLK: CON1.2, IC3.SCLK
- new net N$10: C3.1, IC3.AIN0, IC4.YOUT
- net N$5: now also IC3.AIN1; no longer IC3.AIN0
Other:
- moved on the sheet: R3
Changed lines of the file:
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@@
 <class number="0" name="default" width="0" drill="0">
 </class>
-<class number="1" name="power" width="0.4064" drill="0">
+<class number="1" name="power" width="0.6096" drill="0">
 </class>
 </classes>
@@
 <part name="+3V5" library="supply1" deviceset="+3V3" device=""/>
 <part name="GND8" library="supply1" deviceset="GND" device=""/>
-<part name="FRAME3" library="frames" deviceset="A4L-LOC" device=""/>
-<part name="LED1" library="led" deviceset="LED" device="CHIP-LED0805"/>
+<part name="FRAME3" library="frames" deviceset="A4L-LOC" device="" value="Accelerometer board"/>
+<part name="LED1" library="led" deviceset="LED" device="CHIP-LED0805" value="Power indicator"/>
 <part name="R1" library="rcl" deviceset="R-EU_" device="R0805" value="100R"/>
 <part name="GND9" library="supply1" deviceset="GND" device=""/>
@@
 <part name="C6" library="rcl" deviceset="C-EU" device="C1206K" value="10uF"/>
 <part name="GND2" library="supply1" deviceset="GND" device=""/>
-<part name="CON1" library="con-harting-ml" deviceset="ML6" device=""/>
+<part name="CON1" library="con-harting-ml" deviceset="ML6" device="" value="Main board connector"/>
 <part name="+3V1" library="supply1" deviceset="+3V3" device=""/>
 <part name="GND3" library="supply1" deviceset="GND" device=""/>
@@
 <instance part="R2" gate="G$1" x="182.88" y="106.68" rot="R90"/>
 <instance part="GND11" gate="1" x="182.88" y="96.52"/>
-<instance part="R3" gate="G$1" x="83.82" y="121.92" smashed="yes" rot="R180">
-<attribute name="NAME" x="85.09" y="128.0414" size="1.778" layer="95" rot="R180"/>
-<attribute name="VALUE" x="85.09" y="125.222" size="1.778" layer="96" rot="R180"/>
+<instance part="R3" gate="G$1" x="86.36" y="121.92" smashed="yes" rot="R180">
+<attribute name="NAME" x="87.63" y="128.0414" size="1.778" layer="95" rot="R180"/>
+<attribute name="VALUE" x="87.63" y="125.222" size="1.778" layer="96" rot="R180"/>
 </instance>
 </instances>
@@
 </busses>
 <nets>
-<net name="GND" class="0">
+<net name="GND" class="1">
 <segment>
 <pinref part="IC3" gate="G$1" pin="GND"/>
@@
 </segment>
 </net>
-<net name="+3V3" class="0">
+<net name="+3V3" class="1">
 <segment>
 <pinref part="IC3" gate="G$1" pin="VDD"/>
@@
 <net name="N$5" class="0">
 <segment>
-<pinref part="IC3" gate="G$1" pin="AIN0"/>
-<wire x1="119.38" y1="121.92" x2="149.86" y2="121.92" width="0.1524" layer="91"/>
-<wire x1="149.86" y1="121.92" x2="149.86" y2="124.46" width="0.1524" layer="91"/>
 <pinref part="IC4" gate="G$1" pin="XOUT"/>
-<wire x1="149.86" y1="124.46" x2="160.02" y2="124.46" width="0.1524" layer="91"/>
 <pinref part="C4" gate="G$1" pin="1"/>
 <wire x1="160.02" y1="124.46" x2="185.42" y2="124.46" width="0.1524" layer="91"/>
 <wire x1="160.02" y1="109.22" x2="160.02" y2="124.46" width="0.1524" layer="91"/>
-<junction x="160.02" y="124.46"/>
-</segment>
-</net>
-<net name="N$6" class="0">
-<segment>
-<pinref part="IC4" gate="G$1" pin="YOUT"/>
-<wire x1="185.42" y1="119.38" x2="170.18" y2="119.38" width="0.1524" layer="91"/>
-<wire x1="170.18" y1="119.38" x2="152.4" y2="119.38" width="0.1524" layer="91"/>
-<wire x1="152.4" y1="119.38" x2="152.4" y2="116.84" width="0.1524" layer="91"/>
 <pinref part="IC3" gate="G$1" pin="AIN1"/>
 <wire x1="152.4" y1="116.84" x2="119.38" y2="116.84" width="0.1524" layer="91"/>
-<pinref part="C3" gate="G$1" pin="1"/>
-<wire x1="170.18" y1="119.38" x2="170.18" y2="109.22" width="0.1524" layer="91"/>
-<junction x="170.18" y="119.38"/>
+<wire x1="160.02" y1="124.46" x2="152.4" y2="124.46" width="0.1524" layer="91"/>
+<wire x1="152.4" y1="124.46" x2="152.4" y2="116.84" width="0.1524" layer="91"/>
+<junction x="160.02" y="124.46"/>
 </segment>
 </net>
@@
 </segment>
 </net>
-<net name="N$1" class="0">
-<segment>
+<net name="ADC_CS" class="0">
+<segment>
+<pinref part="IC3" gate="G$1" pin="!CS"/>
+<pinref part="CON1" gate="1" pin="4"/>
+<wire x1="40.64" y1="119.38" x2="38.1" y2="119.38" width="0.1524" layer="91"/>
+<wire x1="38.1" y1="119.38" x2="38.1" y2="129.54" width="0.1524" layer="91"/>
+<wire x1="38.1" y1="129.54" x2="93.98" y2="129.54" width="0.1524" layer="91"/>
+<label x="38.1" y="129.54" size="1.778" layer="95"/>
+</segment>
+</net>
+<net name="ADC_DOUT" class="0">
+<segment>
+<pinref part="R3" gate="G$1" pin="2"/>
+<wire x1="78.74" y1="121.92" x2="81.28" y2="121.92" width="0.1524" layer="91"/>
 <pinref part="CON1" gate="1" pin="1"/>
-<wire x1="55.88" y1="116.84" x2="66.04" y2="116.84" width="0.1524" layer="91"/>
-<wire x1="66.04" y1="116.84" x2="66.04" y2="129.54" width="0.1524" layer="91"/>
-<pinref part="IC3" gate="G$1" pin="!CS"/>
-<wire x1="66.04" y1="129.54" x2="93.98" y2="129.54" width="0.1524" layer="91"/>
-</segment>
-</net>
-<net name="N$2" class="0">
-<segment>
-<pinref part="CON1" gate="1" pin="2"/>
-<wire x1="40.64" y1="116.84" x2="38.1" y2="116.84" width="0.1524" layer="91"/>
-<wire x1="38.1" y1="116.84" x2="38.1" y2="111.76" width="0.1524" layer="91"/>
-<wire x1="38.1" y1="111.76" x2="73.66" y2="111.76" width="0.1524" layer="91"/>
-<wire x1="73.66" y1="111.76" x2="73.66" y2="121.92" width="0.1524" layer="91"/>
-<pinref part="R3" gate="G$1" pin="2"/>
-<wire x1="73.66" y1="121.92" x2="78.74" y2="121.92" width="0.1524" layer="91"/>
-</segment>
-</net>
-<net name="N$3" class="0">
+<wire x1="55.88" y1="116.84" x2="78.74" y2="116.84" width="0.1524" layer="91"/>
+<wire x1="78.74" y1="116.84" x2="78.74" y2="121.92" width="0.1524" layer="91"/>
+<label x="60.96" y="116.84" size="1.778" layer="95"/>
+</segment>
+</net>
+<net name="ADC_DIN" class="0">
 <segment>
 <pinref part="CON1" gate="1" pin="3"/>
@@
 <pinref part="IC3" gate="G$1" pin="DIN"/>
 <wire x1="88.9" y1="116.84" x2="93.98" y2="116.84" width="0.1524" layer="91"/>
-</segment>
-</net>
-<net name="N$4" class="0">
-<segment>
-<pinref part="CON1" gate="1" pin="4"/>
-<wire x1="40.64" y1="119.38" x2="35.56" y2="119.38" width="0.1524" layer="91"/>
-<wire x1="35.56" y1="119.38" x2="35.56" y2="109.22" width="0.1524" layer="91"/>
+<label x="60.96" y="119.38" size="1.778" layer="95"/>
+</segment>
+</net>
+<net name="ADC_SCLK" class="0">
+<segment>
 <pinref part="IC3" gate="G$1" pin="SCLK"/>
-<wire x1="35.56" y1="109.22" x2="93.98" y2="109.22" width="0.1524" layer="91"/>
+<wire x1="38.1" y1="109.22" x2="93.98" y2="109.22" width="0.1524" layer="91"/>
+<wire x1="38.1" y1="109.22" x2="38.1" y2="116.84" width="0.1524" layer="91"/>
+<pinref part="CON1" gate="1" pin="2"/>
+<wire x1="38.1" y1="116.84" x2="40.64" y2="116.84" width="0.1524" layer="91"/>
+<label x="38.1" y="106.68" size="1.778" layer="95"/>
 </segment>
 </net>
@@
 <pinref part="R3" gate="G$1" pin="1"/>
 <pinref part="IC3" gate="G$1" pin="DOUT"/>
-<wire x1="88.9" y1="121.92" x2="93.98" y2="121.92" width="0.1524" layer="91"/>
+<wire x1="91.44" y1="121.92" x2="93.98" y2="121.92" width="0.1524" layer="91"/>
+</segment>
+</net>
+<net name="N$10" class="0">
+<segment>
+<pinref part="IC3" gate="G$1" pin="AIN0"/>
+<wire x1="119.38" y1="121.92" x2="149.86" y2="121.92" width="0.1524" layer="91"/>
+<wire x1="149.86" y1="121.92" x2="149.86" y2="119.38" width="0.1524" layer="91"/>
+<pinref part="IC4" gate="G$1" pin="YOUT"/>
+<wire x1="185.42" y1="119.38" x2="170.18" y2="119.38" width="0.1524" layer="91"/>
+<wire x1="170.18" y1="119.38" x2="149.86" y2="119.38" width="0.1524" layer="91"/>
+<pinref part="C3" gate="G$1" pin="1"/>
+<wire x1="170.18" y1="119.38" x2="170.18" y2="109.22" width="0.1524" layer="91"/>
+<junction x="170.18" y="119.38"/>
 </segment>
 </net>
@@
 </sheet>
 </sheets>
+<errors>
+</errors>
 </schematic>
 </drawing>

Commit message: Final PCB
Parts:
- renumbered IC3 to IC1, IC4 to IC2
Other:
- note removed: "Dual mode: ADC range 0 - Vdd"
- note removed: "OBS. the impedance from the source device into the ADC affects AC perfomance see page 12, when making lowpass filter"
- note removed: "Terminering seriel eller parallel? Max 35cm kabel"
- note removed: "Tjek at connector PCB layout passer"
Changed lines of the file:
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@@
 </classes>
 <parts>
-<part name="IC3" library="tobylib" deviceset="AD7887BRZ" device=""/>
-<part name="IC4" library="tobylib" deviceset="ADXL203CE" device=""/>
+<part name="IC1" library="tobylib" deviceset="AD7887BRZ" device=""/>
+<part name="IC2" library="tobylib" deviceset="ADXL203CE" device=""/>
 <part name="+3V4" library="supply1" deviceset="+3V3" device=""/>
 <part name="GND7" library="supply1" deviceset="GND" device=""/>
@@
 <sheet>
 <plain>
-<text x="48.26" y="160.02" size="1.778" layer="91">Dual mode: ADC range 0 - Vdd</text>
-<text x="48.26" y="162.56" size="1.778" layer="91">OBS. the impedance from the source device into the ADC affects AC perfomance see page 12, when making lowpass filter</text>
-<text x="48.26" y="157.48" size="1.778" layer="91">Tjek at connector PCB layout passer</text>
-<text x="55.88" y="132.08" size="1.778" layer="91">Terminering seriel eller parallel?
-Max 35cm kabel</text>
 <text x="160.02" y="127" size="1.778" layer="91">fc =2.2KHz </text>
 </plain>
 <instances>
-<instance part="IC3" gate="G$1" x="106.68" y="119.38"/>
-<instance part="IC4" gate="G$1" x="198.12" y="119.38"/>
+<instance part="IC1" gate="G$1" x="106.68" y="119.38"/>
+<instance part="IC2" gate="G$1" x="198.12" y="119.38"/>
 <instance part="+3V4" gate="G$1" x="129.54" y="139.7"/>
 <instance part="GND7" gate="1" x="121.92" y="96.52"/>
@@
 <net name="GND" class="1">
 <segment>
-<pinref part="IC3" gate="G$1" pin="GND"/>
+<pinref part="IC1" gate="G$1" pin="GND"/>
 <pinref part="GND7" gate="1" pin="GND"/>
 <wire x1="119.38" y1="109.22" x2="121.92" y2="109.22" width="0.1524" layer="91"/>
@@
 </segment>
 <segment>
-<pinref part="IC4" gate="G$1" pin="GND"/>
+<pinref part="IC2" gate="G$1" pin="GND"/>
 <pinref part="GND8" gate="1" pin="GND"/>
 <wire x1="210.82" y1="109.22" x2="213.36" y2="109.22" width="0.1524" layer="91"/>
@@
 <net name="+3V3" class="1">
 <segment>
-<pinref part="IC3" gate="G$1" pin="VDD"/>
+<pinref part="IC1" gate="G$1" pin="VDD"/>
 <pinref part="+3V4" gate="G$1" pin="+3V3"/>
 <wire x1="119.38" y1="129.54" x2="129.54" y2="129.54" width="0.1524" layer="91"/>
@@
 </segment>
 <segment>
-<pinref part="IC4" gate="G$1" pin="VDD"/>
+<pinref part="IC2" gate="G$1" pin="VDD"/>
 <pinref part="+3V5" gate="G$1" pin="+3V3"/>
 <wire x1="210.82" y1="129.54" x2="220.98" y2="129.54" width="0.1524" layer="91"/>
@@
 <net name="N$5" class="0">
 <segment>
-<pinref part="IC4" gate="G$1" pin="XOUT"/>
+<pinref part="IC2" gate="G$1" pin="XOUT"/>
 <pinref part="C4" gate="G$1" pin="1"/>
 <wire x1="160.02" y1="124.46" x2="185.42" y2="124.46" width="0.1524" layer="91"/>
 <wire x1="160.02" y1="109.22" x2="160.02" y2="124.46" width="0.1524" layer="91"/>
-<pinref part="IC3" gate="G$1" pin="AIN1"/>
+<pinref part="IC1" gate="G$1" pin="AIN1"/>
 <wire x1="152.4" y1="116.84" x2="119.38" y2="116.84" width="0.1524" layer="91"/>
 <wire x1="160.02" y1="124.46" x2="152.4" y2="124.46" width="0.1524" layer="91"/>
@@
 <net name="ADC_CS" class="0">
 <segment>
-<pinref part="IC3" gate="G$1" pin="!CS"/>
+<pinref part="IC1" gate="G$1" pin="!CS"/>
 <pinref part="CON1" gate="1" pin="4"/>
 <wire x1="40.64" y1="119.38" x2="38.1" y2="119.38" width="0.1524" layer="91"/>
@@
 <wire x1="55.88" y1="119.38" x2="88.9" y2="119.38" width="0.1524" layer="91"/>
 <wire x1="88.9" y1="119.38" x2="88.9" y2="116.84" width="0.1524" layer="91"/>
-<pinref part="IC3" gate="G$1" pin="DIN"/>
+<pinref part="IC1" gate="G$1" pin="DIN"/>
 <wire x1="88.9" y1="116.84" x2="93.98" y2="116.84" width="0.1524" layer="91"/>
 <label x="60.96" y="119.38" size="1.778" layer="95"/>
@@
 <net name="ADC_SCLK" class="0">
 <segment>
-<pinref part="IC3" gate="G$1" pin="SCLK"/>
+<pinref part="IC1" gate="G$1" pin="SCLK"/>
 <wire x1="38.1" y1="109.22" x2="93.98" y2="109.22" width="0.1524" layer="91"/>
 <wire x1="38.1" y1="109.22" x2="38.1" y2="116.84" width="0.1524" layer="91"/>
@@
 <net name="N$8" class="0">
 <segment>
-<pinref part="IC4" gate="G$1" pin="ST"/>
+<pinref part="IC2" gate="G$1" pin="ST"/>
 <pinref part="R2" gate="G$1" pin="2"/>
 <wire x1="185.42" y1="114.3" x2="182.88" y2="114.3" width="0.1524" layer="91"/>
@@
 <segment>
 <pinref part="R3" gate="G$1" pin="1"/>
-<pinref part="IC3" gate="G$1" pin="DOUT"/>
+<pinref part="IC1" gate="G$1" pin="DOUT"/>
 <wire x1="91.44" y1="121.92" x2="93.98" y2="121.92" width="0.1524" layer="91"/>
 </segment>
@@
 <net name="N$10" class="0">
 <segment>
-<pinref part="IC3" gate="G$1" pin="AIN0"/>
+<pinref part="IC1" gate="G$1" pin="AIN0"/>
 <wire x1="119.38" y1="121.92" x2="149.86" y2="121.92" width="0.1524" layer="91"/>
 <wire x1="149.86" y1="121.92" x2="149.86" y2="119.38" width="0.1524" layer="91"/>
-<pinref part="IC4" gate="G$1" pin="YOUT"/>
+<pinref part="IC2" gate="G$1" pin="YOUT"/>
 <wire x1="185.42" y1="119.38" x2="170.18" y2="119.38" width="0.1524" layer="91"/>
 <wire x1="170.18" y1="119.38" x2="149.86" y2="119.38" width="0.1524" layer="91"/>
@@
 </schematic>
 </drawing>
-<compatibility>
-<note version="6.3" minversion="6.2.2" severity="warning">
-Since Version 6.2.2 text objects can contain more than one line,
-which will not be processed correctly with this version.
-</note>
-</compatibility>
 </eagle>
